Commit message: mostly working

File: xacro/biped.xacro (robot description, xacro)
@@ -1,4 +1,5 @@
 <?xml version="1.0"?>
-<robot name ="biped" xmlns:xacro="http://www.ros.org/wiki/xacro">
+<robot name ="biped"
+  xmlns:xacro="http://www.ros.org/wiki/xacro">
   <xacro:property name = "foot_width" value = "0.05"/>
   <xacro:property name = "foot_height" value = "0.005"/>
@@ -8,58 +9,78 @@
   <xacro:property name = "lower_leg_length" value = "0.20"/>
   <material name="body">
-      <color rgba="0.5 0.5 0.3 0.7"/>
+    <color rgba="0.5 0.5 0.3 0.7"/>
   </material>
+  <link name="base_link"></link>
   <link name="left_foot">
-  		<inertial>
-	  		<origin xyz="0 0 0" rpy="0 0.0 0.0"/>
-  	  		<mass value="2.043"/>
-	  		<inertia ixx="0.03" ixy="0.0" ixz="0.0" iyy="0.03" iyz="0.0" izz="0.03"/>
-		</inertial>
-		<visual>
-	  		<origin xyz="0 0 ${foot_height/2}" rpy="0 0.0 0.0"/>
-            <geometry>
-              <box size="${foot_length} ${foot_width} ${foot_height}" />
-            </geometry>
-            <material name = "foot">
-            <color rgba="0.7 0 0 0.7"/>
-            </material>
-   		</visual>
-		<collision>
-	  		<origin xyz="0 0 ${foot_height/2}" rpy="0 0.0 0.0"/>
-            <geometry>
-              <box size="${foot_length} ${foot_width} ${foot_height}" />
-            </geometry>
-			<contact_coefficients kd="1.0" kp="1000.0" mu="0"/>
-		</collision>
+    <inertial>
+      <origin xyz="0 0 0" rpy="0 0.0 0.0"/>
+      <mass value="2.043"/>
+      <inertia ixx="0.03" ixy="0.0" ixz="0.0" iyy="0.03" iyz="0.0" izz="0.03"/>
+    </inertial>
+    <visual>
+      <origin xyz="0 0 ${foot_height/2}" rpy="0 0.0 0.0"/>
+      <geometry>
+        <box size="${foot_length} ${foot_width} ${foot_height}" />
+      </geometry>
+      <material name = "foot">
+        <color rgba="0.7 0 0 0.7"/>
+      </material>
+    </visual>
+    <collision>
+      <origin xyz="0 0 ${foot_height/2}" rpy="0 0.0 0.0"/>
+      <geometry>
+        <box size="${foot_length} ${foot_width} ${foot_height}" />
+      </geometry>
+      <contact_coefficients kd="1.0" kp="1000.0" mu="0"/>
+    </collision>
   </link>
   <link name = "lower_left_leg">
-  		<inertial>
-	  		<origin xyz="0 0 ${lower_leg_length/2}"  rpy="0 ${-pi/2} 0.0"/>
-  	  		<mass value="2.043"/>
-	  		<inertia ixx="0.03" ixy="0.0" ixz="0.0" iyy="0.03" iyz="0.0" izz="0.03"/>
-		</inertial>
-		<visual>
-	  		<origin xyz="0 0 ${lower_leg_length/2}"  rpy="0 ${-pi/2} 0.0"/>
-            <geometry>
-              <box size="${lower_leg_length} ${lower_leg_width} ${lower_leg_height}" />
-            </geometry>
-            <material name="leg">
-            <color rgba="0.7 0 0 0.7"/>
-            </material>
-   		</visual>
-		<collision>
-	  		<origin xyz="0 0 ${lower_leg_length/2}"  rpy="0 ${-pi/2} 0.0"/>
-            <geometry>
-              <box size="${lower_leg_length} ${lower_leg_width} ${lower_leg_height}" />
-            </geometry>
-			<contact_coefficients kd="1.0" kp="1000.0" mu="0"/>
-		</collision>
+    <inertial>
+      <origin xyz="0 0 ${lower_leg_length/2}" rpy="0 ${-pi/2} 0.0"/>
+      <mass value="2.043"/>
+      <inertia ixx="0.03" ixy="0.0" ixz="0.0" iyy="0.03" iyz="0.0" izz="0.03"/>
+    </inertial>
+    <visual>
+      <origin xyz="0 0 ${lower_leg_length/2}" rpy="0 ${-pi/2} 0.0"/>
+      <geometry>
+        <box size="${lower_leg_length} ${lower_leg_width} ${lower_leg_height}" />
+      </geometry>
+      <material name="leg">
+        <color rgba="0.7 0 0 0.7"/>
+      </material>
+    </visual>
+    <collision>
+      <origin xyz="0 0 ${lower_leg_length/2}" rpy="0 ${-pi/2} 0.0"/>
+      <geometry>
+        <box size="${lower_leg_length} ${lower_leg_width} ${lower_leg_height}" />
+      </geometry>
+      <contact_coefficients kd="1.0" kp="1000.0" mu="0"/>
+    </collision>
   </link>
+  <joint name="base_joint" type="fixed">
+    <parent link="base_link"/>
+    <child link="lower_left_leg"/>
+  </joint>
   <joint name = "left_ankle" type = "revolute">
-     <axis xyz="0 0 0"/>
-     <limit effort="1000.0" lower="0" upper="2" velocity="0.5"/>
-     <origin rpy="0 0 0" xyz="0 0 0"/>
-     <parent link="lower_left_leg"/>
-     <child link="left_foot"/>
+    <axis xyz="0 0 0"/>
+    <limit effort="1000.0" lower="0" upper="2" velocity="0.5"/>
+    <origin rpy="0 0 0" xyz="0 0 0"/>
+    <parent link="lower_left_leg"/>
+    <child link="left_foot"/>
   </joint>
+  <gazebo>
+    <plugin name="gazebo_ros_control" filename="libgazebo_ros_control.so">
+      <robotNamespace>/biped</robotNamespace>
+    </plugin>
+  </gazebo>
+  <transmission name="left_ankle_transmission">
+    <type>transmission_interface/SimpleTransmission</type>
+    <joint name="left_ankle">
+      <hardwareInterface>hardware_interface/EffortJointInterface</hardwareInterface>
+    </joint>
+    <actuator name="left_ankle_motor">
+      <hardwareInterface>hardware_interface/EffortJointInterface</hardwareInterface>
+      <mechanicalReduction>1</mechanicalReduction>
+    </actuator>
+  </transmission>
 </robot>

Commit message: Works in RVIS, colors

File: xacro/biped.xacro (robot description, xacro)
@@ -63,5 +63,5 @@
   </joint>
   <joint name = "left_ankle" type = "revolute">
-    <axis xyz="0 0 0"/>
+    <axis xyz="0 1 0"/>
     <limit effort="1000.0" lower="0" upper="2" velocity="0.5"/>
     <origin rpy="0 0 0" xyz="0 0 0"/>
@@ -73,4 +73,14 @@
       <robotNamespace>/biped</robotNamespace>
     </plugin>
+  </gazebo>
+  <!--
+    Gazebo colors from
+    https://github.com/osrf/gazebo/blob/master/media/materials/scripts/gazebo.material
+  -->
+  <gazebo reference="left_foot">
+    <material>Gazebo/RedTransparent</material>
+  </gazebo>
+  <gazebo reference="lower_left_leg">
+    <material>Gazebo/RedTransparent</material>
   </gazebo>
   <transmission name="left_ankle_transmission">

Commit message: knee working

File: xacro/biped.xacro (robot description, xacro)
@@ -8,9 +8,82 @@
   <xacro:property name = "lower_leg_height" value = "0.02"/>
   <xacro:property name = "lower_leg_length" value = "0.20"/>
+  <xacro:property name = "upper_leg_width" value = "0.01"/>
+  <xacro:property name = "upper_leg_height" value = "0.02"/>
+  <xacro:property name = "upper_leg_length" value = "0.20"/>
+  <xacro:property name = "motor_length" value = "0.05"/>
+  <xacro:property name = "motor_radius" value = "0.025"/>
   <material name="body">
     <color rgba="0.5 0.5 0.3 0.7"/>
   </material>
   <link name="base_link"></link>
-  <link name="left_foot">
+  <link name = "upper_left_leg">
+    <inertial>
+      <origin xyz="0 0 0" rpy="0 ${-pi/2} 0.0"/>
+      <mass value="2.043"/>
+      <inertia ixx="0.03" ixy="0.0" ixz="0.0" iyy="0.03" iyz="0.0" izz="0.03"/>
+    </inertial>
+    <visual>
+      <origin xyz="0 0 0" rpy="0 ${-pi/2} 0.0"/>
+      <geometry>
+        <box size="${upper_leg_length} ${upper_leg_width} ${upper_leg_height}" />
+      </geometry>
+      <material name="leg">
+        <color rgba="0.7 0 0 0.7"/>
+      </material>
+    </visual>
+    <collision>
+      <origin xyz="0 0 0" rpy="0 ${-pi/2} 0.0"/>
+      <geometry>
+        <box size="${upper_leg_length} ${upper_leg_width} ${upper_leg_height}" />
+      </geometry>
+      <contact_coefficients kd="1.0" kp="1000.0" mu="0"/>
+    </collision>
+  </link>
+<link name="left_knee_motor">
+   <inertial>
+     <origin xyz="0 0 0" rpy="0 0 0"/>
+     <mass value="1"/>
+     <inertia ixx="100"  ixy="0"  ixz="0" iyy="100" iyz="0" izz="100" />
+   </inertial>
+   <visual>
+     <origin xyz="0 0 0" rpy="${pi/2} 0 0" />
+     <geometry>
+       <cylinder radius="${motor_radius}" length="${motor_length}"/>
+     </geometry>
+     <material name="Cyan">
+       <color rgba="0 1.0 1.0 1.0"/>
+     </material>
+   </visual>
+   <collision>
+     <origin xyz="0 0 0" rpy="0 0 0"/>
+     <geometry>
+       <cylinder radius="0.1" length="0.1"/>
+     </geometry>
+   </collision>
+ </link>
+  <link name = "lower_left_leg">
+    <inertial>
+      <origin xyz="0 0 ${-lower_leg_length/2}" rpy="0 ${-pi/2} 0.0"/>
+      <mass value="2.043"/>
+      <inertia ixx="0.03" ixy="0.0" ixz="0.0" iyy="0.03" iyz="0.0" izz="0.03"/>
+    </inertial>
+    <visual>
+      <origin xyz="0 0 ${-lower_leg_length/2}" rpy="0 ${-pi/2} 0.0"/>
+      <geometry>
+        <box size="${lower_leg_length} ${lower_leg_width} ${lower_leg_height}" />
+      </geometry>
+      <material name="lleg">
+        <color rgba="0 0.7 0 0.7"/>
+      </material>
+    </visual>
+    <collision>
+      <origin xyz="0 0 ${-lower_leg_length/2}" rpy="0 ${-pi/2} 0.0"/>
+      <geometry>
+        <box size="${lower_leg_length} ${lower_leg_width} ${lower_leg_height}" />
+      </geometry>
+      <contact_coefficients kd="1.0" kp="1000.0" mu="0"/>
+    </collision>
+  </link>
+    <link name="left_foot">
     <inertial>
       <origin xyz="0 0 0" rpy="0 0.0 0.0"/>
@@ -19,5 +92,5 @@
     </inertial>
     <visual>
-      <origin xyz="0 0 ${foot_height/2}" rpy="0 0.0 0.0"/>
+      <origin xyz="0 0 ${-motor_radius -foot_height/2}" rpy="0 0.0 0.0"/>
       <geometry>
         <box size="${foot_length} ${foot_width} ${foot_height}" />
@@ -28,5 +101,5 @@
     </visual>
     <collision>
-      <origin xyz="0 0 ${foot_height/2}" rpy="0 0.0 0.0"/>
+      <origin xyz="0 0 0" rpy="0 0.0 0.0"/>
       <geometry>
         <box size="${foot_length} ${foot_width} ${foot_height}" />
@@ -35,30 +108,46 @@
     </collision>
   </link>
-  <link name = "lower_left_leg">
-    <inertial>
-      <origin xyz="0 0 ${lower_leg_length/2}" rpy="0 ${-pi/2} 0.0"/>
-      <mass value="2.043"/>
-      <inertia ixx="0.03" ixy="0.0" ixz="0.0" iyy="0.03" iyz="0.0" izz="0.03"/>
-    </inertial>
-    <visual>
-      <origin xyz="0 0 ${lower_leg_length/2}" rpy="0 ${-pi/2} 0.0"/>
-      <geometry>
-        <box size="${lower_leg_length} ${lower_leg_width} ${lower_leg_height}" />
-      </geometry>
-      <material name="leg">
-        <color rgba="0.7 0 0 0.7"/>
-      </material>
-    </visual>
-    <collision>
-      <origin xyz="0 0 ${lower_leg_length/2}" rpy="0 ${-pi/2} 0.0"/>
-      <geometry>
-        <box size="${lower_leg_length} ${lower_leg_width} ${lower_leg_height}" />
-      </geometry>
-      <contact_coefficients kd="1.0" kp="1000.0" mu="0"/>
-    </collision>
-  </link>
+ <link name="left_ankle_motor">
+   <inertial>
+     <origin xyz="0 0 0" rpy="0 0 0"/>
+     <mass value="1"/>
+     <inertia ixx="100"  ixy="0"  ixz="0" iyy="100" iyz="0" izz="100" />
+   </inertial>
+   <visual>
+     <origin xyz="0 0 0" rpy="${pi/2} 0 0" />
+     <geometry>
+       <cylinder radius="${motor_radius}" length="${motor_length}"/>
+     </geometry>
+     <material name="Cyan">
+       <color rgba="0 1.0 1.0 1.0"/>
+     </material>
+   </visual>
+   <collision>
+     <origin xyz="0 0 0" rpy="0 0 0"/>
+     <geometry>
+       <cylinder radius="0.1" length="0.1"/>
+     </geometry>
+   </collision>
+ </link>
   <joint name="base_joint" type="fixed">
     <parent link="base_link"/>
+    <child link="upper_left_leg"/>
+  </joint>
+  <joint name="upper_left_leg_to_knee_motor_joint" type="fixed">
+    <parent link="upper_left_leg"/>
+    <origin xyz="0 0 ${-upper_leg_length/2}" rpy="0 0 0"/>
+    <child link="left_knee_motor"/>
+  </joint>
+  <joint name = "left_knee" type = "revolute">
+    <axis xyz="0 1 0"/>
+    <limit effort="1000.0" lower="0" upper="2" velocity="0.5"/>
+    <origin rpy="0 0 0" xyz="0 0 0"/>
+    <parent link="left_knee_motor"/>
     <child link="lower_left_leg"/>
+  </joint>
+  <joint name = "lower_left_leg_to_ankle_motor" type="fixed">
+     <parent link = "lower_left_leg"/>
+     <child link = "left_ankle_motor"/>
+     <origin xyz="0 0 ${-lower_leg_length} "/>
   </joint>
   <joint name = "left_ankle" type = "revolute">
@@ -66,5 +155,5 @@
     <limit effort="1000.0" lower="0" upper="2" velocity="0.5"/>
     <origin rpy="0 0 0" xyz="0 0 0"/>
-    <parent link="lower_left_leg"/>
+    <parent link="left_ankle_motor"/>
     <child link="left_foot"/>
   </joint>
@@ -82,5 +171,8 @@
   </gazebo>
   <gazebo reference="lower_left_leg">
-    <material>Gazebo/RedTransparent</material>
+    <material>Gazebo/Gold</material>
+  </gazebo>
+  <gazebo reference="upper_left_leg">
+    <material>Gazebo/Red</material>
   </gazebo>
   <transmission name="left_ankle_transmission">
@@ -94,3 +186,13 @@
     </actuator>
   </transmission>
+  <transmission name="left_knee_transmission">
+    <type>transmission_interface/SimpleTransmission</type>
+    <joint name="left_knee">
+      <hardwareInterface>hardware_interface/EffortJointInterface</hardwareInterface>
+    </joint>
+    <actuator name="left_knee_motor">
+      <hardwareInterface>hardware_interface/EffortJointInterface</hardwareInterface>
+      <mechanicalReduction>1</mechanicalReduction>
+    </actuator>
+  </transmission>
 </robot>

Commit message: Decrease moments to make sim move better

File: xacro/biped.xacro (robot description, xacro)
@@ -42,7 +42,7 @@
 <link name="left_knee_motor">
    <inertial>
-     <origin xyz="0 0 0" rpy="0 0 0"/>
+     <origin xyz="0 0 0" rpy="${pi/2} 0 0" />
      <mass value="1"/>
-     <inertia ixx="100"  ixy="0"  ixz="0" iyy="100" iyz="0" izz="100" />
+     <inertia ixx="0.03"  ixy="0"  ixz="0" iyy="0.03" iyz="0" izz="0.03" />
    </inertial>
    <visual>
@@ -56,7 +56,7 @@
    </visual>
    <collision>
-     <origin xyz="0 0 0" rpy="0 0 0"/>
+     <origin xyz="0 0 0" rpy="${pi/2} 0 0" />
      <geometry>
-       <cylinder radius="0.1" length="0.1"/>
+       <cylinder radius="${motor_radius}" length="${motor_length}"/>
      </geometry>
    </collision>
@@ -87,5 +87,5 @@
     <link name="left_foot">
     <inertial>
-      <origin xyz="0 0 0" rpy="0 0.0 0.0"/>
+      <origin xyz="0 0 ${-motor_radius -foot_height/2}" rpy="0 0.0 0.0"/>
       <mass value="2.043"/>
       <inertia ixx="0.03" ixy="0.0" ixz="0.0" iyy="0.03" iyz="0.0" izz="0.03"/>
@@ -101,5 +101,5 @@
     </visual>
     <collision>
-      <origin xyz="0 0 0" rpy="0 0.0 0.0"/>
+      <origin xyz="0 0 ${-motor_radius -foot_height/2}" rpy="0 0.0 0.0"/>
       <geometry>
         <box size="${foot_length} ${foot_width} ${foot_height}" />
@@ -112,5 +112,5 @@
      <origin xyz="0 0 0" rpy="0 0 0"/>
      <mass value="1"/>
-     <inertia ixx="100"  ixy="0"  ixz="0" iyy="100" iyz="0" izz="100" />
+     <inertia ixx="0.03"  ixy="0"  ixz="0" iyy="0.03" iyz="0" izz="0.03" />
    </inertial>
    <visual>
@@ -124,7 +124,7 @@
    </visual>
    <collision>
-     <origin xyz="0 0 0" rpy="0 0 0"/>
+     <origin xyz="0 0 0" rpy="${pi/2} 0 0" />
      <geometry>
-       <cylinder radius="0.1" length="0.1"/>
+       <cylinder radius="${motor_radius}" length="${motor_length}"/>
      </geometry>
    </collision>
@@ -141,5 +141,5 @@
   <joint name = "left_knee" type = "revolute">
     <axis xyz="0 1 0"/>
-    <limit effort="1000.0" lower="0" upper="2" velocity="0.5"/>
+    <limit effort="1000.0" lower="-2" upper="2" velocity="0.5"/>
     <origin rpy="0 0 0" xyz="0 0 0"/>
     <parent link="left_knee_motor"/>
@@ -153,5 +153,5 @@
   <joint name = "left_ankle" type = "revolute">
     <axis xyz="0 1 0"/>
-    <limit effort="1000.0" lower="0" upper="2" velocity="0.5"/>
+    <limit effort="1000.0" lower="-2" upper="2" velocity="0.5"/>
     <origin rpy="0 0 0" xyz="0 0 0"/>
     <parent link="left_ankle_motor"/>

Commit message: Box link

File: xacro/biped.xacro (robot description, xacro)
@@ -17,27 +17,28 @@
   </material>
   <link name="base_link"></link>
-  <link name = "upper_left_leg">
-    <inertial>
-      <origin xyz="0 0 0" rpy="0 ${-pi/2} 0.0"/>
-      <mass value="2.043"/>
-      <inertia ixx="0.03" ixy="0.0" ixz="0.0" iyy="0.03" iyz="0.0" izz="0.03"/>
-    </inertial>
-    <visual>
-      <origin xyz="0 0 0" rpy="0 ${-pi/2} 0.0"/>
-      <geometry>
-        <box size="${upper_leg_length} ${upper_leg_width} ${upper_leg_height}" />
-      </geometry>
-      <material name="leg">
-        <color rgba="0.7 0 0 0.7"/>
-      </material>
-    </visual>
-    <collision>
-      <origin xyz="0 0 0" rpy="0 ${-pi/2} 0.0"/>
-      <geometry>
-        <box size="${upper_leg_length} ${upper_leg_width} ${upper_leg_height}" />
-      </geometry>
-      <contact_coefficients kd="1.0" kp="1000.0" mu="0"/>
-    </collision>
-  </link>
+  <xacro:macro name="box_link" params="name m x y z origin:='0 0 0' rpy:='0 0 0' color">
+    <link name = "${name}">
+      <inertial>
+        <origin xyz="${origin}" rpy="${rpy}"/>
+        <mass value="${m}"/>
+        <inertia ixx = "${m/12*(y*y+z*z)}" ixy = "0.0" ixz="0.0" iyy="${m/12*(x*x+z*z)}" iyz="0.0" izz="${m/12*(x*x+y*y)}"/>
+      </inertial>
+      <visual>
+        <origin xyz="${origin}" rpy="${rpy}"/>
+        <geometry>
+          <box size="${x} ${y} ${z}" />
+        </geometry>
+        <material name="${name}_material">
+          <color rgba = "${color}"/>
+        </material>
+      </visual>
+      <collision>
+        <origin xyz="${origin}" rpy="${rpy}"/>
+        <geometry>
+          <box size="${x} ${y} ${z}" />
+        </geometry>
+      </collision>
+    </link>
+  </xacro:macro>
 <link name="left_knee_motor">
    <inertial>
@@ -62,4 +63,7 @@
    </collision>
  </link>
+ <xacro:box_link name="upper_left_leg" x="${upper_leg_length}" y="${upper_leg_height}" z="${upper_leg_width}" m = "1"  origin="0 0 ${-upper_leg_length/2}" rpy="0 ${-pi/2} 0.0" color = "0 0.7 0 0.7"/>
+ <xacro:box_link name="lower_left_leg" x="${lower_leg_length}" y="${lower_leg_height}" z="${lower_leg_width}" m = "1" origin="0 0 ${-lower_leg_length/2}" rpy="0 ${-pi/2} 0.0" color = "0 0.7 0 0.7"/>
+<!--
   <link name = "lower_left_leg">
     <inertial>
@@ -80,9 +84,10 @@
       <origin xyz="0 0 ${-lower_leg_length/2}" rpy="0 ${-pi/2} 0.0"/>
       <geometry>
-        <box size="${lower_leg_length} ${lower_leg_width} ${lower_leg_height}" />
+        <box size="${lower_leg_length} ${lower_leg_width} ${lower_leg_height}" />b
       </geometry>
       <contact_coefficients kd="1.0" kp="1000.0" mu="0"/>
     </collision>
   </link>
+-->
     <link name="left_foot">
     <inertial>
@@ -136,5 +141,5 @@
   <joint name="upper_left_leg_to_knee_motor_joint" type="fixed">
     <parent link="upper_left_leg"/>
-    <origin xyz="0 0 ${-upper_leg_length/2}" rpy="0 0 0"/>
+    <origin xyz="0 0 ${-upper_leg_length}" rpy="0 0 0"/>
     <child link="left_knee_motor"/>
   </joint>
