Commit message: Cleaned up with macros

File: xacro/biped.xacro (robot description, xacro)
@@ -2,4 +2,7 @@
 <robot name ="biped"
   xmlns:xacro="http://www.ros.org/wiki/xacro">
+  <!--
+    Properties
+  -->
   <xacro:property name = "foot_width" value = "0.05"/>
   <xacro:property name = "foot_height" value = "0.005"/>
@@ -13,8 +16,10 @@
   <xacro:property name = "motor_length" value = "0.05"/>
   <xacro:property name = "motor_radius" value = "0.025"/>
-  <material name="body">
-    <color rgba="0.5 0.5 0.3 0.7"/>
-  </material>
-  <link name="base_link"></link>
+  <xacro:property name = "color_red" value = "1 0 0 1"/>
+  <xacro:property name = "color_gold" value = "0.831 0.686 0.216 1"/>
+  <xacro:property name = "color_dark_grey" value = "0.4 0.4 0.4 1"/>
+  <!--
+    Macros
+  -->
   <xacro:macro name="box_link" params="name m x y z origin:='0 0 0' rpy:='0 0 0' color">
     <link name = "${name}">
@@ -41,98 +46,40 @@
     </link>
   </xacro:macro>
-<link name="left_knee_motor">
-   <inertial>
-     <origin xyz="0 0 0" rpy="${pi/2} 0 0" />
-     <mass value="1"/>
-     <inertia ixx="0.03"  ixy="0"  ixz="0" iyy="0.03" iyz="0" izz="0.03" />
-   </inertial>
-   <visual>
-     <origin xyz="0 0 0" rpy="${pi/2} 0 0" />
-     <geometry>
-       <cylinder radius="${motor_radius}" length="${motor_length}"/>
-     </geometry>
-     <material name="Cyan">
-       <color rgba="0 1.0 1.0 1.0"/>
-     </material>
-   </visual>
-   <collision>
-     <origin xyz="0 0 0" rpy="${pi/2} 0 0" />
-     <geometry>
-       <cylinder radius="${motor_radius}" length="${motor_length}"/>
-     </geometry>
-   </collision>
- </link>
- <xacro:box_link name="upper_left_leg" x="${upper_leg_length}" y="${upper_leg_height}" z="${upper_leg_width}" m = "1"  origin="0 0 ${-upper_leg_length/2}" rpy="0 ${-pi/2} 0.0" color = "0 0.7 0 0.7"/>
- <xacro:box_link name="lower_left_leg" x="${lower_leg_length}" y="${lower_leg_height}" z="${lower_leg_width}" m = "1" origin="0 0 ${-lower_leg_length/2}" rpy="0 ${-pi/2} 0.0" color = "0 0.7 0 0.7"/>
-<!--
-  <link name = "lower_left_leg">
-    <inertial>
-      <origin xyz="0 0 ${-lower_leg_length/2}" rpy="0 ${-pi/2} 0.0"/>
-      <mass value="2.043"/>
-      <inertia ixx="0.03" ixy="0.0" ixz="0.0" iyy="0.03" iyz="0.0" izz="0.03"/>
-    </inertial>
-    <visual>
-      <origin xyz="0 0 ${-lower_leg_length/2}" rpy="0 ${-pi/2} 0.0"/>
-      <geometry>
-        <box size="${lower_leg_length} ${lower_leg_width} ${lower_leg_height}" />
-      </geometry>
-      <material name="lleg">
-        <color rgba="0 0.7 0 0.7"/>
-      </material>
-    </visual>
-    <collision>
-      <origin xyz="0 0 ${-lower_leg_length/2}" rpy="0 ${-pi/2} 0.0"/>
-      <geometry>
-        <box size="${lower_leg_length} ${lower_leg_width} ${lower_leg_height}" />b
-      </geometry>
-      <contact_coefficients kd="1.0" kp="1000.0" mu="0"/>
-    </collision>
-  </link>
--->
-    <link name="left_foot">
-    <inertial>
-      <origin xyz="0 0 ${-motor_radius -foot_height/2}" rpy="0 0.0 0.0"/>
-      <mass value="2.043"/>
-      <inertia ixx="0.03" ixy="0.0" ixz="0.0" iyy="0.03" iyz="0.0" izz="0.03"/>
-    </inertial>
-    <visual>
-      <origin xyz="0 0 ${-motor_radius -foot_height/2}" rpy="0 0.0 0.0"/>
-      <geometry>
-        <box size="${foot_length} ${foot_width} ${foot_height}" />
-      </geometry>
-      <material name = "foot">
-        <color rgba="0.7 0 0 0.7"/>
-      </material>
-    </visual>
-    <collision>
-      <origin xyz="0 0 ${-motor_radius -foot_height/2}" rpy="0 0.0 0.0"/>
-      <geometry>
-        <box size="${foot_length} ${foot_width} ${foot_height}" />
-      </geometry>
-      <contact_coefficients kd="1.0" kp="1000.0" mu="0"/>
-    </collision>
-  </link>
- <link name="left_ankle_motor">
-   <inertial>
-     <origin xyz="0 0 0" rpy="0 0 0"/>
-     <mass value="1"/>
-     <inertia ixx="0.03"  ixy="0"  ixz="0" iyy="0.03" iyz="0" izz="0.03" />
-   </inertial>
-   <visual>
-     <origin xyz="0 0 0" rpy="${pi/2} 0 0" />
-     <geometry>
-       <cylinder radius="${motor_radius}" length="${motor_length}"/>
-     </geometry>
-     <material name="Cyan">
-       <color rgba="0 1.0 1.0 1.0"/>
-     </material>
-   </visual>
-   <collision>
-     <origin xyz="0 0 0" rpy="${pi/2} 0 0" />
-     <geometry>
-       <cylinder radius="${motor_radius}" length="${motor_length}"/>
-     </geometry>
-   </collision>
- </link>
+  <xacro:macro name="cylinder_link" params="name r l m color origin:='0 0 0' rpy:='0 0 0' ">
+    <link name="${name}">
+      <inertial>
+        <origin xyz="${origin}" rpy="${rpy}" />
+        <mass value="${m}"/>
+        <inertia ixx="${m*r*r/4+m*l*l}" ixy="0" ixz="0" iyy="${m*r*r/4+m*l*l}" iyz="0" izz="${m*r*r/2}" />
+      </inertial>
+      <visual>
+        <origin xyz="${origin}" rpy="${rpy}" />
+        <geometry>
+          <cylinder radius="${r}" length="${l}"/>
+        </geometry>
+        <material name="${name}_color">
+          <color rgba="${color}"/>
+        </material>
+      </visual>
+      <collision>
+        <origin xyz="${origin}" rpy="${rpy}" />
+        <geometry>
+          <cylinder radius="${r}" length="${l}"/>
+        </geometry>
+      </collision>
+    </link>
+  </xacro:macro>
+  <!--
+    Links
+  -->
+  <link name="base_link"></link>
+  <xacro:cylinder_link name="left_knee_motor" m="1" r="${motor_radius}" l="${motor_length}" rpy="${pi/2} 0 0" color="${color_dark_grey}"/>
+  <xacro:box_link name="upper_left_leg" x="${upper_leg_length}" y="${upper_leg_height}" z="${upper_leg_width}" m = "1" origin="0 0 ${-upper_leg_length/2}" rpy="0 ${-pi/2} 0.0" color = "${color_red}"/>
+  <xacro:box_link name="lower_left_leg" x="${lower_leg_length}" y="${lower_leg_height}" z="${lower_leg_width}" m = "1" origin="0 0 ${-lower_leg_length/2}" rpy="0 ${-pi/2} 0.0" color = "${color_gold}"/>
+  <xacro:cylinder_link name="left_ankle_motor" m="1" r="${motor_radius}" l="${motor_length}" rpy="${pi/2} 0 0" color="${color_dark_grey}"/>
+  <xacro:box_link name="left_foot" x="${foot_length}" y="${foot_width}" z="${foot_height}" m = "20" origin="0 0 ${-motor_radius -foot_height/2}" rpy="0 0.0 0.0" color = "${color_gold}"/>
+  <!--
+    Joints
+  -->
   <joint name="base_joint" type="fixed">
     <parent link="base_link"/>
@@ -152,7 +99,7 @@
   </joint>
   <joint name = "lower_left_leg_to_ankle_motor" type="fixed">
-     <parent link = "lower_left_leg"/>
-     <child link = "left_ankle_motor"/>
-     <origin xyz="0 0 ${-lower_leg_length} "/>
+    <parent link = "lower_left_leg"/>
+    <child link = "left_ankle_motor"/>
+    <origin xyz="0 0 ${-lower_leg_length} "/>
   </joint>
   <joint name = "left_ankle" type = "revolute">
@@ -163,9 +110,4 @@
     <child link="left_foot"/>
   </joint>
-  <gazebo>
-    <plugin name="gazebo_ros_control" filename="libgazebo_ros_control.so">
-      <robotNamespace>/biped</robotNamespace>
-    </plugin>
-  </gazebo>
   <!--
     Gazebo colors from
@@ -181,4 +123,21 @@
     <material>Gazebo/Red</material>
   </gazebo>
+  <gazebo reference="left_knee_motor">
+    <material>Gazebo/DarkGray</material>
+  </gazebo>
+  <gazebo reference="left_ankle_motor">
+    <material>Gazebo/DarkGray</material>
+  </gazebo>
+  <!--
+    Gazebo ros control
+  -->
+  <gazebo>
+    <plugin name="gazebo_ros_control" filename="libgazebo_ros_control.so">
+      <robotNamespace>/biped</robotNamespace>
+    </plugin>
+  </gazebo>
+  <!--
+    Transmissions for robot control
+  -->
   <transmission name="left_ankle_transmission">
     <type>transmission_interface/SimpleTransmission</type>

Commit message: Extended range of motion

File: xacro/biped.xacro (robot description, xacro)
@@ -93,5 +93,5 @@
   <joint name = "left_knee" type = "revolute">
     <axis xyz="0 1 0"/>
-    <limit effort="1000.0" lower="-2" upper="2" velocity="0.5"/>
+    <limit effort="1000.0" lower="${-2*pi}" upper="${2*pi}" velocity="0.5"/>
     <origin rpy="0 0 0" xyz="0 0 0"/>
     <parent link="left_knee_motor"/>
@@ -105,5 +105,5 @@
   <joint name = "left_ankle" type = "revolute">
     <axis xyz="0 1 0"/>
-    <limit effort="1000.0" lower="-2" upper="2" velocity="0.5"/>
+    <limit effort="1000.0" lower="${-2*pi}" upper="${2*pi}" velocity="0.5"/>
     <origin rpy="0 0 0" xyz="0 0 0"/>
     <parent link="left_ankle_motor"/>

Commit message: Model Mitch's motors

File: xacro/biped.xacro (robot description, xacro)
@@ -8,12 +8,21 @@
   <xacro:property name = "foot_height" value = "0.005"/>
   <xacro:property name = "foot_length" value = "0.1000"/>
+  <xacro:property name = "foot_mass" value = "10"/>
   <xacro:property name = "lower_leg_width" value = "0.01"/>
   <xacro:property name = "lower_leg_height" value = "0.02"/>
   <xacro:property name = "lower_leg_length" value = "0.20"/>
+  <xacro:property name = "lower_leg_mass" value = "0.10"/>
   <xacro:property name = "upper_leg_width" value = "0.01"/>
   <xacro:property name = "upper_leg_height" value = "0.02"/>
   <xacro:property name = "upper_leg_length" value = "0.20"/>
-  <xacro:property name = "motor_length" value = "0.05"/>
-  <xacro:property name = "motor_radius" value = "0.025"/>
+  <xacro:property name = "upper_leg_mass" value = "0.10"/>
+<!--
+  Motor based on RMD-L-4015
+  http://www.gyems.cn/794904.html
+-->
+  <xacro:property name = "motor_length" value = "0.033"/>
+  <xacro:property name = "motor_radius" value = "0.0198"/>
+  <xacro:property name = "motor_mass" value = "0.120"/>
+  <xacro:property name = "motor_torque_nm" value = "0.49"/> <!-- stall torque, nominal is 0.22 -->
   <xacro:property name = "color_red" value = "1 0 0 1"/>
   <xacro:property name = "color_gold" value = "0.831 0.686 0.216 1"/>
@@ -25,5 +34,5 @@
     <link name = "${name}">
       <inertial>
-        <origin xyz="${origin}" rpy="${rpy}"/>
+        <origin xyz="0 0 0" rpy="${rpy}"/>
         <mass value="${m}"/>
         <inertia ixx = "${m/12*(y*y+z*z)}" ixy = "0.0" ixz="0.0" iyy="${m/12*(x*x+z*z)}" iyz="0.0" izz="${m/12*(x*x+y*y)}"/>
@@ -74,9 +83,9 @@
   -->
   <link name="base_link"></link>
-  <xacro:cylinder_link name="left_knee_motor" m="1" r="${motor_radius}" l="${motor_length}" rpy="${pi/2} 0 0" color="${color_dark_grey}"/>
-  <xacro:box_link name="upper_left_leg" x="${upper_leg_length}" y="${upper_leg_height}" z="${upper_leg_width}" m = "1" origin="0 0 ${-upper_leg_length/2}" rpy="0 ${-pi/2} 0.0" color = "${color_red}"/>
-  <xacro:box_link name="lower_left_leg" x="${lower_leg_length}" y="${lower_leg_height}" z="${lower_leg_width}" m = "1" origin="0 0 ${-lower_leg_length/2}" rpy="0 ${-pi/2} 0.0" color = "${color_gold}"/>
-  <xacro:cylinder_link name="left_ankle_motor" m="1" r="${motor_radius}" l="${motor_length}" rpy="${pi/2} 0 0" color="${color_dark_grey}"/>
-  <xacro:box_link name="left_foot" x="${foot_length}" y="${foot_width}" z="${foot_height}" m = "20" origin="0 0 ${-motor_radius -foot_height/2}" rpy="0 0.0 0.0" color = "${color_gold}"/>
+  <xacro:cylinder_link name="left_knee_motor" m="${motor_mass}" r="${motor_radius}" l="${motor_length}" rpy="${pi/2} 0 0" color="${color_dark_grey}"/>
+  <xacro:box_link name="upper_left_leg" x="${upper_leg_length}" y="${upper_leg_height}" z="${upper_leg_width}" m = "${upper_leg_mass}" origin="0 0 ${-upper_leg_length/2}" rpy="0 ${-pi/2} 0.0" color = "${color_red}"/>
+  <xacro:box_link name="lower_left_leg" x="${lower_leg_length}" y="${lower_leg_height}" z="${lower_leg_width}" m = "${lower_leg_mass}" origin="0 0 ${-lower_leg_length/2}" rpy="0 ${-pi/2} 0.0" color = "${color_gold}"/>
+  <xacro:cylinder_link name="left_ankle_motor" m="${motor_mass}" r="${motor_radius}" l="${motor_length}" rpy="${pi/2} 0 0" color="${color_dark_grey}"/>
+  <xacro:box_link name="left_foot" x="${foot_length}" y="${foot_width}" z="${foot_height}" m = "${foot_mass}" origin="0 0 ${-motor_radius -foot_height/2}" rpy="0 0.0 0.0" color = "${color_gold}"/>
   <!--
     Joints
@@ -93,5 +102,5 @@
   <joint name = "left_knee" type = "revolute">
     <axis xyz="0 1 0"/>
-    <limit effort="1000.0" lower="${-2*pi}" upper="${2*pi}" velocity="0.5"/>
+    <limit effort="${motor_torque_nm}" lower="${-2*pi}" upper="${2*pi}" velocity="0.5"/>
     <origin rpy="0 0 0" xyz="0 0 0"/>
     <parent link="left_knee_motor"/>
@@ -105,5 +114,5 @@
   <joint name = "left_ankle" type = "revolute">
     <axis xyz="0 1 0"/>
-    <limit effort="1000.0" lower="${-2*pi}" upper="${2*pi}" velocity="0.5"/>
+    <limit effort="${motor_torque_nm}" lower="${-2*pi}" upper="${2*pi}" velocity="0.5"/>
     <origin rpy="0 0 0" xyz="0 0 0"/>
     <parent link="left_ankle_motor"/>

Commit message: Added the torso.

File: xacro/biped.xacro (robot description, xacro)
@@ -5,4 +5,8 @@
     Properties
   -->
+  <xacro:property name = "torso_width" value = "0.1"/>
+  <xacro:property name = "torso_height" value = "0.15"/>
+  <xacro:property name = "torso_depth" value = "0.05"/>
+  <xacro:property name = "torso_mass" value = "0.2"/>
   <xacro:property name = "foot_width" value = "0.05"/>
   <xacro:property name = "foot_height" value = "0.005"/>
@@ -24,5 +28,5 @@
   <xacro:property name = "motor_radius" value = "0.0198"/>
   <xacro:property name = "motor_mass" value = "0.120"/>
-  <xacro:property name = "motor_torque_nm" value = "0.49"/> <!-- stall torque, nominal is 0.22 -->
+  <xacro:property name = "motor_torque_nm" value = "2.49"/> <!-- stall torque 0.49 , nominal is 0.22 -->
   <xacro:property name = "color_red" value = "1 0 0 1"/>
   <xacro:property name = "color_gold" value = "0.831 0.686 0.216 1"/>
@@ -83,6 +87,8 @@
   -->
   <link name="base_link"></link>
+  <xacro:box_link name="torso" x="${torso_depth}" y="${torso_width}" z="${torso_height}" m = "${torso_mass}" origin="0 0 ${-torso_height/2}" rpy="0 0 0.0" color = "${color_dark_grey}"/>
+  <xacro:cylinder_link name="left_hip_motor" m="${motor_mass}" r="${motor_radius}" l="${motor_length}" rpy="${pi/2} 0 0" color="${color_dark_grey}"/>
+  <xacro:box_link name="upper_left_leg" x="${upper_leg_length}" y="${upper_leg_height}" z="${upper_leg_width}" m = "${upper_leg_mass}" origin="0 0 ${-upper_leg_length/2}" rpy="0 ${-pi/2} 0.0" color = "${color_red}"/>
   <xacro:cylinder_link name="left_knee_motor" m="${motor_mass}" r="${motor_radius}" l="${motor_length}" rpy="${pi/2} 0 0" color="${color_dark_grey}"/>
-  <xacro:box_link name="upper_left_leg" x="${upper_leg_length}" y="${upper_leg_height}" z="${upper_leg_width}" m = "${upper_leg_mass}" origin="0 0 ${-upper_leg_length/2}" rpy="0 ${-pi/2} 0.0" color = "${color_red}"/>
   <xacro:box_link name="lower_left_leg" x="${lower_leg_length}" y="${lower_leg_height}" z="${lower_leg_width}" m = "${lower_leg_mass}" origin="0 0 ${-lower_leg_length/2}" rpy="0 ${-pi/2} 0.0" color = "${color_gold}"/>
   <xacro:cylinder_link name="left_ankle_motor" m="${motor_mass}" r="${motor_radius}" l="${motor_length}" rpy="${pi/2} 0 0" color="${color_dark_grey}"/>
@@ -93,4 +99,16 @@
   <joint name="base_joint" type="fixed">
     <parent link="base_link"/>
+    <child link="torso"/>
+  </joint>
+  <joint name="torso_to_left_hip_motor_joint" type="fixed">
+    <parent link="torso"/>
+    <origin xyz="0 ${-torso_width/2} ${-torso_height}" rpy="0 0 0"/>
+    <child link="left_hip_motor"/>
+  </joint>
+  <joint name = "left_hip" type = "revolute">
+    <axis xyz="0 1 0"/>
+    <limit effort="${motor_torque_nm}" lower="${-2*pi}" upper="${2*pi}" velocity="0.5"/>
+    <origin rpy="0 0 0" xyz="0 0 0"/>
+    <parent link="left_hip_motor"/>
     <child link="upper_left_leg"/>
   </joint>
@@ -114,5 +132,5 @@
   <joint name = "left_ankle" type = "revolute">
     <axis xyz="0 1 0"/>
-    <limit effort="${motor_torque_nm}" lower="${-2*pi}" upper="${2*pi}" velocity="0.5"/>
+    <limit effort="${motor_torque_nm*3}" lower="${-2*pi}" upper="${2*pi}" velocity="0.5"/>
     <origin rpy="0 0 0" xyz="0 0 0"/>
     <parent link="left_ankle_motor"/>
@@ -137,4 +155,10 @@
   <gazebo reference="left_ankle_motor">
     <material>Gazebo/DarkGray</material>
+  </gazebo>
+  <gazebo reference="left_hip_motor">
+    <material>Gazebo/DarkGray</material>
+  </gazebo>
+  <gazebo reference="torso">
+    <material>Gazebo/Gold</material>
   </gazebo>
   <!--
@@ -156,5 +180,5 @@
     <actuator name="left_ankle_motor">
       <hardwareInterface>hardware_interface/EffortJointInterface</hardwareInterface>
-      <mechanicalReduction>1</mechanicalReduction>
+      <mechanicalReduction>3</mechanicalReduction>
     </actuator>
   </transmission>
@@ -169,3 +193,13 @@
     </actuator>
   </transmission>
+  <transmission name="left_hip_transmission">
+    <type>transmission_interface/SimpleTransmission</type>
+    <joint name="left_hip">
+      <hardwareInterface>hardware_interface/EffortJointInterface</hardwareInterface>
+    </joint>
+    <actuator name="left_hip_motor">
+      <hardwareInterface>hardware_interface/EffortJointInterface</hardwareInterface>
+      <mechanicalReduction>1</mechanicalReduction>
+    </actuator>
+  </transmission>
 </robot>
